Commit message: latest

File: mybot_ws/src/mybot_description/urdf/mybot.xacro (robot description, xacro)
@@ -1,8 +1,10 @@
 <?xml version='1.0'?>
 <robot name="myrobot" xmlns:xacro="http://www.ros.org/wiki/xacro">
-  <xacro:include filename="$(find mybot_description)/urdf/mybot.gazebo" />
+  <xacro:arg name="id" default="1" />
+  <xacro:include filename="$(find mybot_description)/urdf/mybot.gazebo"/>
+  <idbridge id="$(arg id)"/>
   <xacro:include filename="$(find mybot_description)/urdf/materials.xacro" />
   <xacro:include filename="$(find mybot_description)/urdf/macros.xacro" />
-  <link name='chassis'>
+  <link name='chassis$(arg id)'>
     <pose>0 0 0.1 0 0 0</pose>
     <inertial>
@@ -15,10 +17,10 @@
       />
     </inertial>
-    <collision name='collision'>
+    <collision name='collision$(arg id)'>
       <geometry>
         <box size=".4 .2 .1"/>
       </geometry>
     </collision>
-    <visual name='chassis_visual'>
+    <visual name='chassis_visual$(arg id)'>
       <origin xyz="0 0 0" rpy=" 0 0 0"/>
       <geometry>
@@ -27,7 +29,7 @@
     </visual>
   </link>
-  <link name="left_wheel">
+  <link name="left_wheel$(arg id)">
     <!--origin xyz="0.1 0.13 0.1" rpy="0 1.5707 1.5707"/-->
-    <collision name="collision">
+    <collision name="collision$(arg id)">
       <origin xyz="0 0 0" rpy="0 1.5707 1.5707"/>
       <geometry>
@@ -43,5 +45,5 @@
       </surface>
     </collision>
-    <visual name="left_wheel_visual">
+    <visual name="left_wheel_visual$(arg id)">
       <origin xyz="0 0 0" rpy="0 1.0 0"/>
       <geometry>
@@ -59,7 +61,7 @@
     </inertial>
   </link>
-<link name="left_wheel_back">
+<link name="left_wheel_back$(arg id)">
     <!--origin xyz="0.1 0.13 0.1" rpy="0 1.5707 1.5707"/-->
-    <collision name="collision">
+    <collision name="collision$(arg id)">
       <origin xyz="0 0 0" rpy="0 1.5707 1.5707"/>
       <geometry>
@@ -75,5 +77,5 @@
       </surface>
     </collision>
-    <visual name="left_wheel_visual">
+    <visual name="left_wheel_visual$(arg id)">
       <origin xyz="0 0 0" rpy="0 1.0 0"/>
       <geometry>
@@ -91,7 +93,7 @@
     </inertial>
   </link>
-  <link name="right_wheel">
+  <link name="right_wheel$(arg id)">
     <!--origin xyz="0.1 -0.13 0.1" rpy="0 1.5707 1.5707"/-->
-    <collision name="collision">
+    <collision name="collision$(arg id)">
       <origin xyz="0 0 0" rpy="0 1.5707 1.5707"/>
       <geometry>
@@ -107,5 +109,5 @@
       </surface>
     </collision>
-    <visual name="right_wheel_visual">
+    <visual name="right_wheel_visual$(arg id)">
       <origin xyz="0 0 0" rpy="0 0 0"/>
       <geometry>
@@ -123,7 +125,7 @@
     </inertial>
   </link>
-<link name="right_wheel_back">
+<link name="right_wheel_back$(arg id)">
     <!--origin xyz="0.1 -0.13 0.1" rpy="0 1.5707 1.5707"/-->
-    <collision name="collision">
+    <collision name="collision$(arg id)">
       <origin xyz="0 0 0" rpy="0 1.5707 1.5707"/>
       <geometry>
@@ -139,5 +141,5 @@
       </surface>
     </collision>
-    <visual name="right_wheel_visual">
+    <visual name="right_wheel_visual$(arg id)">
       <origin xyz="0 0 0" rpy="0 0 0"/>
       <geometry>
@@ -155,32 +157,32 @@
     </inertial>
   </link>
-  <joint type="continuous" name="left_wheel_hinge">
+  <joint type="continuous" name="left_wheel_hinge$(arg id)">
     <origin xyz="0.1 0.151 0" rpy="0 0 0"/>
-    <child link="left_wheel"/>
-    <parent link="chassis"/>
+    <child link="left_wheel$(arg id)"/>
+    <parent link="chassis$(arg id)"/>
     <axis xyz="0 1 0" rpy="0 0 0"/>
     <limit effort="100" velocity="100"/>
     <joint_properties damping="0.0" friction="0.0"/>
   </joint>
-  <joint type="continuous" name="right_wheel_hinge">
+  <joint type="continuous" name="right_wheel_hinge$(arg id)">
     <origin xyz="0.1 -0.151 0" rpy="0 0 0"/>
-    <child link="right_wheel"/>
-    <parent link="chassis"/>
+    <child link="right_wheel$(arg id)"/>
+    <parent link="chassis$(arg id)"/>
     <axis xyz="0 1 0" rpy="0 0 0"/>
     <limit effort="100" velocity="100"/>
     <joint_properties damping="0.0" friction="0.0"/>
   </joint>
-  <joint type="continuous" name="left_wheel_hinge_b">
+  <joint type="continuous" name="left_wheel_hinge_b$(arg id)">
     <origin xyz="-0.15 0.151 0" rpy="0 0 0"/>
-    <child link="left_wheel_back"/>
-    <parent link="chassis"/>
+    <child link="left_wheel_back$(arg id)"/>
+    <parent link="chassis$(arg id)"/>
     <axis xyz="0 1 0" rpy="0 0 0"/>
     <limit effort="100" velocity="100"/>
     <joint_properties damping="0.0" friction="0.0"/>
   </joint>
-  <joint type="continuous" name="right_wheel_hinge_b">
+  <joint type="continuous" name="right_wheel_hinge_b$(arg id)">
     <origin xyz="-0.15 -0.151 0" rpy="0 0 0"/>
-    <child link="right_wheel_back"/>
-    <parent link="chassis"/>
+    <child link="right_wheel_back$(arg id)"/>
+    <parent link="chassis$(arg id)"/>
     <axis xyz="0 1 0" rpy="0 0 0"/>
     <limit effort="100" velocity="100"/>
