Commit message: joystik embbeded

File: bot_new/src/final_plank/urdf/final_plank.urdf (robot description, URDF)
Before this commit: robot final_plank, 3 links, 2 joints
Links:
- added link new_p1; collision box size=.15 6 .04; visual box size=.15 6 .04
- added link new_p2; collision box size=.15 6 .04; visual box size=.15 6 .04
Joints:
- added joint grouding2: type fixed, parent plank, child new_p1, origin xyz=1.38777878078145E-15 0.075 .650000000000009 rpy=0 0 1.5708
- added joint grouding3: type fixed, parent plank, child new_p2, origin xyz=1.38777878078145E-15 0.075 -.050000000000009 rpy=0 0 1.5708
